File: kicad_project/eso32-iot.kicad_sch (KiCad schematic)
At the start: 0 parts

Commit message: update schematic and PCB layout
Parts:
- added C1, C2, C5: 0.1u, symbol Device:C
- added C3, C4: 10u, symbol Device:C_Polarized
- added C6: 1u, symbol Device:C
- added F1: 0ZCH0110AF2E, FUSC3226X100N, symbol 0ZCH0110AF2E:0ZCH0110AF2E
- added J: SS-52400-002, SS-52400-002:BELFUSE_SS-52400-002, symbol SS-52400-002:SS-52400-002
- added J2: B2B-PH-SM4-TB, B2B-PH-SM4-TB:JST_B2B-PH-SM4-TB, symbol B2B-PH-SM4-TB:B2B-PH-SM4-TB
- added LED1, LED4: LTST-C170KRKT, LEDC2012X120N, symbol LTST-C170KRKT:LTST-C170KRKT
- added LED2: LTST-C170GKT, LEDC2012X120N, symbol LTST-C170GKT:LTST-C170GKT
- added LED3: LTST-C170TBKT, LEDC2012X120N, symbol LTST-C170TBKT:LTST-C170TBKT
- added R1, R2: 10k, symbol Device:R
- added R10, R7, R8, R9: 470, symbol Device:R
- added R3, R4: 5k1, symbol Device:R
- added R5: 2k, symbol Device:R
- added R6: 20k, symbol Device:R
- added U1: MCP73871, Package_DFN_QFN:QFN-20-1EP_4x4mm_P0.5mm_EP2.5x2.5mm, symbol Battery_Management:MCP73871
- added VR1: LM1117MPX-3.3, LM1117MPX-3.3:VREG_LM1117MPX-3.3, symbol LM1117MPX-3.3:LM1117MPX-3.3
Connections:
- new net: LED3.1 (K), R9.2
- new net: F1.1, J.B4 (VBUSB1)
- new net: R6.1, U1.12 (PROG3)
- new net: R5.1, U1.13 (PROG1)
- new net: J2.2, R8.1, U1.14 (V_{BAT}), U1.15 (V_{BAT}), U1.16 (V_{BAT_SENSE}), U1.8 (STAT1/~{LBO})
- new net: R2.1, U1.5 (THERM)
- new net: R9.1, U1.6 (~{PG})
- new net: R7.1, U1.7 (STAT2)
- new net: R1.1, U1.9 (~{TE})
- new net: LED2.1 (K), R8.2
- new net: LED1.1 (K), R7.2
- new net: J.A5 (CC1), R4.2
- new net: J.B5 (CC2), R3.2
- new net +3.3V: C4.1, C5.1, LED4.2 (A), VR1.2 (VOUT_2), VR1.4 (VOUT_4)
- new net +5V: C2.1, C3.1, U1.1 (OUT), U1.20 (OUT), VR1.3 (VIN)
- new net +5V_USB: C6.1, F1.2, LED1.2 (A), LED2.2 (A), LED3.2 (A), U1.17 (CE), U1.18 (IN), U1.19 (IN), U1.2 (VPCC), U1.4 (PROG2)
- new net GND: C1.1, C2.2, C3.2, C4.2, C5.2, C6.2, J.A1 (GNDA1), J.A12 (GNDA2), J.B1 (GNDB1), J.B12 (GNDB2), J.G1 (GND/SHIELD), J.G2 (GND/SHIELD), J.G3 (GND/SHIELD), J.G4 (GND/SHIELD), J.S1 (GND/SHIELD), J.S2 (GND/SHIELD), J.S3 (GND/SHIELD), J.S4 (GND/SHIELD), J2.1, R1.2, R10.1, R2.2, R3.1, R4.1, R5.2, R6.2, U1.10 (V_{SS}), U1.11 (V_{SS}), U1.21 (V_{SS}), VR1.1 (GND)
- new net PWD_LED: LED4.1 (K), R10.2
- new net USB_DN: J.A7 (DN1), J.B7 (DN2)
- new net USB_DP: J.A6 (DP1), J.B6 (DP2)
- new net VBUS: J.A4 (VBUSA1)
- no-connect marks 0 -> 10
Other:
- added sheet ESP32-C3-02 (esp32-C3-02.kicad_sch)
- note added: "Battery JST connector"
- note added: "LDO voltage regulator"
- note added: "Lipo battery charger"
- note added: "Power indicator LED"
- note added: "USB-C connector"
- title: (none) -> ESP32 sensor board

Commit message: update schematic and PCB layout
Parts:
- R10: renamed from R6; value 20k -> 20K
- R7: renamed from R1; value 10k -> 10K
- R8: renamed from R2; value 10k -> 10K
- R9: renamed from R5; value 2k -> 2K
- renumbered C2 to C1, C3 to C2, C4 to C3, C5 to C4, C1 to C5, J2 to J1, J to J2, R4 to R1, R3 to R2, R7 to R3, R8 to R4, R9 to R5, R10 to R6
Connections:
- net at J1.2, R4.1, U1.14 (V_{BAT})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: now also R5.1, U1.6 (~{PG})
- net CHARGING_POWER_GOOD: now reaches R3.1, U1.7 (STAT2)
Other:
- sheet ESP32-C3-02 ports: added USB_DN, USB_DP, VBUS; removed none
