File: kicad_project/eso32-iot.kicad_sch (KiCad schematic)
At the start: 25 parts, among them J1 B2B-PH-SM4-TB, J2 SS-52400-002, U1 MCP73871

Commit message: update schematic and PCB layout
Parts:
- J1: footprint B2B-PH-SM4-TB:JST_B2B-PH-SM4-TB -> Footprints:JST_B2B-PH-SM4-TB
- J2: footprint SS-52400-002:BELFUSE_SS-52400-002 -> Footprints:BELFUSE_SS-52400-002
- VR1: footprint LM1117MPX-3.3:VREG_LM1117MPX-3.3 -> Footprints:VREG_LM1117MPX-3.3
Changed lines of the file:
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@@
 			)
 		)
-		(property "Footprint" "B2B-PH-SM4-TB:JST_B2B-PH-SM4-TB"
+		(property "Footprint" "Footprints:JST_B2B-PH-SM4-TB"
 			(at 33.02 156.21 0)
 			(hide yes)
@@
 			)
 		)
-		(property "Footprint" "SS-52400-002:BELFUSE_SS-52400-002"
+		(property "Footprint" "Footprints:BELFUSE_SS-52400-002"
 			(at 58.42 49.53 0)
 			(hide yes)
@@
 			)
 		)
-		(property "Footprint" "LM1117MPX-3.3:VREG_LM1117MPX-3.3"
+		(property "Footprint" "Footprints:VREG_LM1117MPX-3.3"
 			(at 48.26 119.38 0)
 			(hide yes)

Commit message: update schematic and PCB layout
Changed lines of the file:
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@@
 	(wire
 		(pts
-			(xy 38.1 156.21) (xy 46.99 156.21)
+			(xy 38.1 156.21) (xy 48.26 156.21)
 		)
 		(stroke
@@
 		)
 	)
+	(label "VBAT"
+		(at 48.26 156.21 0)
+		(effects
+			(font
+				(size 1.27 1.27)
+			)
+			(justify left bottom)
+		)
+	)
 	(label ""
 		(at 180.34 49.53 0)
@@
 		(effects
 			(font
-				(size 1.27 1.27)
-			)
-			(justify left bottom)
-		)
-	)
-	(label "VBAT"
-		(at 46.99 156.21 0)
-		(effects
-			(font
