File: kicad_project/esp32-C3-02.kicad_sch (KiCad schematic)
At the start: 0 parts

Commit message: update schematic and PCB layout
Parts:
- added C7: 1u, symbol Device:C
- added C8: C, symbol Device:C
- added C9: C_Polarized, symbol Device:C_Polarized
- added J3: GSD090012SEU, GSD090012SEU:AMPHENOL_GSD090012SEU, symbol GSD090012SEU:GSD090012SEU
- added R11: 22K1, symbol Device:R
- added R12: 47K5, symbol Device:R
- added R13: 1K, symbol Device:R
- added U2: W25Q32JVSSIQ, W25Q32JVSSIQ:SOIC127P790X216-8N, symbol W25Q32JVSSIQ:W25Q32JVSSIQ
- added U3: USBLC6-2SC6, Package_TO_SOT_SMD:SOT-23-6, symbol Power_Protection:USBLC6-2SC6
- added U4: CP2102N-Axx-xQFN20, Package_DFN_QFN:SiliconLabs_QFN-20-1EP_3x3mm_P0.5mm, symbol Interface_USB:CP2102N-Axx-xQFN20
- added U5: ESP32-C3-WROOM-02-H4, ESP32-C3-WROOM-02-H4:MODULE_ESP32-C3-WROOM-02-H4, symbol ESP32-C3-WROOM-02-H4:ESP32-C3-WROOM-02-H4
Connections:
- new net: J3.G1 (SHIELD_GND), J3.G2 (SHIELD_GND), J3.G3 (SHIELD_GND), J3.G4 (SHIELD_GND)
- new net: U4.12 (GND), U4.21 (GND), U4.3 (GND)
- new net: R13.1, U4.6 (VDD), U4.7 (VREGIN)
- new net: C7.1, R11.2, R12.1, U4.8 (VBUS)
- new net: R13.2, U4.9 (~{RST})
- new net: U5.19 (GND), U5.20 (GND), U5.21 (GND), U5.22 (GND), U5.23 (GND), U5.24 (GND), U5.25 (GND), U5.26 (GND), U5.27 (GND), U5.28 (GND), U5.29 (GND), U5.30 (GND), U5.31 (GND), U5.32 (GND), U5.33 (GND), U5.34 (GND), U5.35 (GND), U5.36 (GND), U5.37 (GND), U5.38 (GND), U5.39 (GND), U5.9 (GND)
- new net GND: C7.2, R12.2, U3.2 (GND)
- new net USB_D+: U3.3 (I/O2), U4.4 (D+)
- new net USB_D-: U3.1 (I/O1), U4.5 (D-)
- new net VBUS: R11.1, U3.5 (VBUS)

Commit message: update schematic and PCB layout
Parts:
- added C12, C7: 10u, symbol Device:C_Polarized
- added C13, C14, C8: 0.1u, symbol Device:C
- added LED5: LTST-C170GKT, LEDC2012X120N, symbol LTST-C170GKT:LTST-C170GKT
- added LED6: LTST-C170TBKT, LEDC2012X120N, symbol LTST-C170TBKT:LTST-C170TBKT
- added R14, R18, R20: 470, symbol Device:R
- added R15, R16, R22: 50, symbol Device:R
- added R19: 10K, symbol Device:R
- added TP1: Test MOSI, symbol Connector:TestPoint
- added TP2: Test MISO, symbol Connector:TestPoint
- added TP3: Test SCLK, symbol Connector:TestPoint
- added TP4: Test CS_SD, symbol Connector:TestPoint
- added TP5: Test CS, symbol Connector:TestPoint
- C10: renamed from C8; value C -> 0.1u
- C9: value C_Polarized -> 4.7u
- renumbered C7 to C11, U5 to U3, U3 to U5
Connections:
- net GND: now also C10.1, C9.2, J3.3 (VSS1), J3.6 (VSS2), J3.8 (DAT1), J3.9 (DAT2), J3.G1 (SHIELD_GND), J3.G2 (SHIELD_GND), J3.G3 (SHIELD_GND), J3.G4 (SHIELD_GND), U2.4 (GND), U3.19 (GND), U3.20 (GND), U3.21 (GND), U3.22 (GND), U3.23 (GND), U3.24 (GND), U3.25 (GND), U3.26 (GND), U3.27 (GND), U3.28 (GND), U3.29 (GND), U3.30 (GND), U3.31 (GND), U3.32 (GND), U3.33 (GND), U3.34 (GND), U3.35 (GND), U3.36 (GND), U3.37 (GND), U3.38 (GND), U3.39 (GND), U3.9 (GND), U4.12 (GND), U4.21 (GND), U4.3 (GND), C12.2, C13.2, C14.2, C7.2, C8.2
- net CS_SD: now reaches J3.1 (CD/DAT3)
- net CS_SD: now also R19.1, TP4.1
- net MOSI_DI: now reaches J3.2 (CMD)
- net MOSI_DI: now also U2.5 (DI(IO0)), R15.2, TP1.1
- net at J3.4 (VDD1): now also C12.1, C13.1
- net SCLK: now reaches J3.5 (CLK)
- net SCLK: now also U2.6 (CLK), R20.1, TP3.1
- net at J3.7 (DAT0): now also R16.1
- net CS: now reaches U2.1 (~{CS})
- net CS: now also U3.10 (IO10), TP5.1
- net at U2.2 (DO(IO1)): now also R22.2
- net +3.3V: now reaches U2.3 (~{WP}(IO2))
- net +3.3V: now also C10.2, C9.1, R13.1, U2.7 (~{HOLD}/~{RESET}(IO3)), U2.8 (VCC), U3.1 (3V3), U4.6 (VDD), U4.7 (VREGIN), C14.1, C7.1, C8.1, LED5.2 (A), LED6.2 (A), R19.2
- net DTS: now reaches U4.15 (~{CTS})
- net RTX: now reaches U4.16 (~{RTS})
- net RX_TX: now reaches U4.17 (RXD)
- net RX_TX: now also U3.12 (TXD)
- net TX_RX: now reaches U4.18 (TXD)
- net TX_RX: now also U3.11 (RXD)
- net at U4.19 (~{RXT}/GPIO.3): now also R18.1
- net at U4.20 (~{TXT}/GPIO.2): now also R14.1
- net GPIO18: now reaches U3.13 (IO18)
- net GPIO19: now reaches U3.14 (IO19)
- net SCL: now reaches U3.15 (IO3)
- net MISO_DO: now reaches U3.16 (IO2)
- net MISO_DO: now also R16.2, R22.1, TP2.1
- net PHOTO_C: now reaches U3.17 (IO1)
- net CD_SD: now reaches U3.18 (IO0)
- net EN: now reaches U3.2 (EN)
- net SDA: now reaches U3.3 (IO4)
- net MIC_OUT: now reaches U3.4 (IO5)
- net at U3.5 (IO6): now also R20.2
- net at U3.6 (IO7): now also R15.1
- net GPIO8: now reaches U3.7 (IO8)
- net BOOT: now reaches U3.8 (IO9)
- new net: LED6.1 (K), R18.2
- new net: LED5.1 (K), R14.2
- no-connect marks 0 -> 7
Other:
- added sheet Sensors (sensors.kicad_sch)
- added sheet User Inteterface (user_interface.kicad_sch)
- note added: "ESP32-C3-02"
- note added: "Flash memory"
- note added: "SD card module"
- note added: "USB module"
- title: (none) -> ESP32 C3 USB. and flash memory
- moved on the sheet: C10, C11, C9, J3, R11, R12, R13, U2, U3, U4, U5

Commit message: Update schematic and PCB layout
Other:
- sheet Sensors ports: added MIC_OUT, PHOTO_C, SCL, SDA; removed none
Changed lines of the file:
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@@
 	(wire
 		(pts
+			(xy 149.86 139.7) (xy 158.75 139.7)
+		)
+		(stroke
+			(width 0)
+			(type default)
+		)
+	)
+	(wire
+		(pts
 			(xy 36.83 77.47) (xy 27.94 77.47)
 		)
@@
 	(wire
 		(pts
+			(xy 149.86 143.51) (xy 158.75 143.51)
+		)
+		(stroke
+			(width 0)
+			(type default)
+		)
+	)
+	(wire
+		(pts
 			(xy 266.7 40.64) (xy 270.51 40.64)
 		)
@@
 	(wire
 		(pts
+			(xy 149.86 130.81) (xy 158.75 130.81)
+		)
+		(stroke
+			(width 0)
+			(type default)
+		)
+	)
+	(wire
+		(pts
 			(xy 140.97 85.09) (xy 140.97 97.79)
 		)
@@
 	(wire
 		(pts
+			(xy 149.86 134.62) (xy 158.75 134.62)
+		)
+		(stroke
+			(width 0)
+			(type default)
+		)
+	)
+	(wire
+		(pts
 			(xy 27.94 77.47) (xy 27.94 80.01)
 		)
@@
 			)
 		)
+		(pin "MIC_OUT" input
+			(at 149.86 130.81 0)
+			(effects
+				(font
+					(size 1.27 1.27)
+				)
+				(justify right)
+			)
+		)
+		(pin "PHOTO_C" input
+			(at 149.86 134.62 0)
+			(effects
+				(font
+					(size 1.27 1.27)
+				)
+				(justify right)
+			)
+		)
+		(pin "SCL" input
+			(at 149.86 139.7 0)
+			(effects
+				(font
+					(size 1.27 1.27)
+				)
+				(justify right)
+			)
+		)
+		(pin "SDA" input
+			(at 149.86 143.51 0)
+			(effects
+				(font
+					(size 1.27 1.27)
+				)
+				(justify right)
+			)
+		)
