File: kicad_project/esp32-C3-02.kicad_sch (KiCad schematic)
At the start: 30 parts, among them J3 GSD090012SEU, U2 W25Q32JVSSIQ, U3 ESP32-C3-WROOM-02-H4, U4 CP2102N-Axx-xQFN20, U5 USBLC6-2SC6

Commit message: update schematic and PCB layout
Parts:
- J3: footprint GSD090012SEU:AMPHENOL_GSD090012SEU -> Footprints:AMPHENOL_GSD090012SEU
- U2: footprint W25Q32JVSSIQ:SOIC127P790X216-8N -> Footprints:SOIC127P790X216-8N
- U3: footprint ESP32-C3-WROOM-02-H4:MODULE_ESP32-C3-WROOM-02-H4 -> Footprints:MODULE_ESP32-C3-WROOM-02-H4
- U4: footprint Package_DFN_QFN:SiliconLabs_QFN-20-1EP_3x3mm_P0.5mm -> Footprints:QFN50P400X400X100-21N
Changed lines of the file:
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@@
 			)
 		)
-		(property "Footprint" "GSD090012SEU:AMPHENOL_GSD090012SEU"
+		(property "Footprint" "Footprints:AMPHENOL_GSD090012SEU"
 			(at 217.17 123.19 0)
 			(hide yes)
@@
 			)
 		)
-		(property "Footprint" "W25Q32JVSSIQ:SOIC127P790X216-8N"
+		(property "Footprint" "Footprints:SOIC127P790X216-8N"
 			(at 60.96 143.51 0)
 			(hide yes)
@@
 			)
 		)
-		(property "Footprint" "Package_DFN_QFN:SiliconLabs_QFN-20-1EP_3x3mm_P0.5mm"
+		(property "Footprint" "Footprints:QFN50P400X400X100-21N"
 			(at 107.95 104.14 0)
 			(hide yes)
@@
 			)
 		)
-		(property "Footprint" "ESP32-C3-WROOM-02-H4:MODULE_ESP32-C3-WROOM-02-H4"
+		(property "Footprint" "Footprints:MODULE_ESP32-C3-WROOM-02-H4"
 			(at 217.17 54.61 0)
 			(hide yes)

Commit message: update schematic and PCB layout
Connections:
- net RTX renamed RTS
Changed lines of the file:
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@@
 		)
 	)
-	(label "RTX"
+	(label "RTS"
 		(at 88.9 59.69 0)
 		(effects
@@
 		)
 	)
-	(label "RTX"
+	(label "RTS"
 		(at 156.21 165.1 0)
 		(effects
