File: kicad_project/sensors.kicad_sch (KiCad schematic)
At the start: 0 parts

Commit message: Update schematic and PCB layout
Parts:
- added C15, C16, C18, C20: 0.1u, symbol Device:C
- added MK1: CMC-5042PF-AC, CMC-5042PF-AC:CUI_CMC-5042PF-AC, symbol CMC-5042PF-AC:CMC-5042PF-AC
- added Q1: TEMT6000X01, TEMT6000X01:TRANS_TEMT6000X01, symbol TEMT6000X01:TEMT6000X01
- added R23, R30: 10K, symbol Device:R
- added R24, R25: 4K7, symbol Device:R
- added R26, R28: 2K, symbol Device:R
- added R27, R29: 1M, symbol Device:R
- added R31: 100K, symbol Device:R
- added U6: BME280, BME280:PSON65P250X250X100-8N, symbol BME280:BME280
- added U7: MAX4466EXK, MAX4466EXK:SOT65P210X110-5N, symbol MAX4466EXK:MAX4466EXK
Connections:
- new net: C16.1, R26.2, R28.1
- new net: MK1.OUT, R27.2, R28.2, R29.1, U7.1 (IN+)
- new net +3.3V: C15.1, C18.1, R23.1, R24.1, R25.1, R26.1, R27.1, U6.2 (CSB), U6.6 (VDDIO), U6.8 (VDD), U7.5 (VCC)
- new net GND: C15.2, C16.2, C18.2, C20.1, MK1.GND, Q1.1, R29.2, R30.1, R30.2, R31.2, U6.1 (GND), U6.5 (SDO), U6.7 (GND), U7.2 (GND), U7.3 (IN-)
- new net MIC_OUT: C20.2, R31.1, U7.4 (OUT)
- new net PHOTO_C: Q1.3, R23.2
- new net SCL: R24.2, U6.4 (SCK)
- new net SDA: R25.2, U6.3 (SDI)
