File: kicad_project/sensors.kicad_sch (KiCad schematic)
At the start: 17 parts, among them Q1 TEMT6000X01, U6 BME280, U7 MAX4466EXK

Commit message: update schematic and PCB layout
Parts:
- MK1: footprint CMC-5042PF-AC:CUI_CMC-5042PF-AC -> Footprints:CUI_CMC-5042PF-AC
- Q1: footprint TEMT6000X01:TRANS_TEMT6000X01 -> Footprints:TRANS_TEMT6000X01
- U6: footprint BME280:PSON65P250X250X100-8N -> Footprints:PSON65P250X250X100-8N
- U7: footprint MAX4466EXK:SOT65P210X110-5N -> Footprints:SOT65P210X110-5N
Changed lines of the file:
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@@
 			)
 		)
-		(property "Footprint" "CMC-5042PF-AC:CUI_CMC-5042PF-AC"
+		(property "Footprint" "Footprints:CUI_CMC-5042PF-AC"
 			(at 49.53 128.27 0)
 			(hide yes)
@@
 			)
 		)
-		(property "Footprint" "BME280:PSON65P250X250X100-8N"
+		(property "Footprint" "Footprints:PSON65P250X250X100-8N"
 			(at 77.47 49.53 0)
 			(hide yes)
@@
 			)
 		)
-		(property "Footprint" "TEMT6000X01:TRANS_TEMT6000X01"
+		(property "Footprint" "Footprints:TRANS_TEMT6000X01"
 			(at 153.67 49.53 0)
 			(hide yes)
@@
 			)
 		)
-		(property "Footprint" "MAX4466EXK:SOT65P210X110-5N"
+		(property "Footprint" "Footprints:SOT65P210X110-5N"
 			(at 109.22 128.27 0)
 			(hide yes)
