File: kicad_project/user_interface.kicad_sch (KiCad schematic)
At the start: 0 parts

Commit message: Update schematic and PCB layout
Parts:
- added C21: 0.1u, symbol Device:C
- added C22: 1u, symbol Device:C
- added J4: Conn_01x04_Pin, symbol Connector:Conn_01x04_Pin
- added Q2, Q3: BC817, Package_TO_SOT_SMD:SOT-23, symbol Transistor_BJT:BC817
- added R32, R33, R34: 10K, symbol Device:R
- added S1, S2: USLPT2819DT2TR, USLPT2819DT2TR:SW_USLPT2819DT2TR, symbol USLPT2819DT2TR:USLPT2819DT2TR
Connections:
- new net: Q2.1 (B), R33.2
- new net: Q3.1 (B), R34.2
- new net +3.3V: J4.1 (Pin_1), R32.1
- new net BOOT: C21.1, Q3.2 (E), S1.3, S1.4
- new net DTR: Q3.3 (C), R33.1
- new net EN: C22.1, Q2.3 (C), R32.2, S2.3, S2.4
- new net GND: C21.2, C22.2, J4.4 (Pin_4), S1.1, S1.2, S2.1, S2.2
- new net RTS: Q2.2 (E), R34.1
