File: kicad_project/eso32-iot.kicad_pcb (KiCad board)
At the start: 4 copper layers, 83 parts, among them J1 B2B-PH-SM4-TB, J2 SS-52400-002, J3 GSD090012SEU, J4 Conn_01x04_Pin, J5 Conn_01x05_Pin, Q1 TEMT6000X01, Q2 BC817, Q3 BC817, U1 MCP73871, U2 W25Q32JVSSIQ, U3 ESP32-C3-WROOM-02-H4, U4 CP2102N-Axx-xQFN20, U5 USBLC6-2SC6, U6 BME280, U7 MAX4466EXK

Commit message: update schematic and PCB layout
Parts:
- moved J3 155.5 mm to (236.0, 151.8)
- moved C9 152.8 mm to (26.4, 34.3), turned to 180 degrees
- moved U5 151.5 mm to (24.9, 26.0), turned to 90 degrees
- moved U3 151.4 mm to (256.0, 108.9)
- moved LED5 144.2 mm to (39.2, 29.6), turned to 90 degrees
- moved LED6 143.2 mm to (41.8, 29.6), turned to 90 degrees
- moved R11 142.3 mm to (26.7, 30.7), turned to -90 degrees
- moved R12 139.4 mm to (30.7, 30.7), turned to -90 degrees
- moved R13 138.5 mm to (32.7, 30.7), turned to 90 degrees
- moved R10 138.4 mm to (30.4, 156.6)
- moved R4 138.4 mm to (26.0, 153.7)
- moved R5 138.4 mm to (26.0, 156.6)
- moved R7 138.4 mm to (30.4, 147.8)
- moved R9 138.4 mm to (30.4, 153.7)
- moved C6 138.4 mm to (39.6, 153.9)
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
Commit message: update schematic and PCB layout
Parts:
- moved LED1 46.9 mm to (81.9, 143.8)
- moved LED2 46.9 mm to (81.9, 147.2)
- moved LED3 46.9 mm to (81.9, 150.6)
- moved R10 46.9 mm to (77.3, 155.4)
- moved R7 46.9 mm to (77.3, 146.6)
- moved R8 46.9 mm to (77.3, 149.6)
- moved R9 46.9 mm to (77.3, 152.5)
- moved C6 46.9 mm to (86.5, 152.7)
- moved R3 46.9 mm to (72.9, 149.6)
- moved R4 46.9 mm to (72.9, 152.5)
- moved R5 46.9 mm to (72.9, 155.4)
- moved U1 46.9 mm to (74.2, 160.1)
- moved C7 45.3 mm to (200.2, 86.1)
- moved C8 45.3 mm to (201.4, 89.8)
- moved R15 45.3 mm to (201.5, 97.1)
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