File: eso32-iot/esp32-C3-02.kicad_sch (KiCad schematic)
At the start: 30 parts, among them J3 GSD090012SEU, U2 W25Q32JVSSIQ, U3 ESP32-C3-WROOM-02-H4, U4 CP2102N-Axx-xQFN20, U5 USBLC6-2SC6

Commit message: Update schematic and PCB layout
Changed lines of the file:
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@@
-		)
-	)
-	(label "PHOTO_C"
-		(at 158.75 134.62 0)
-		(effects
-			(font
-				(size 1.27 1.27)
-			)
-			(justify left bottom)
 		)
 	)
 	(label "DTS"
 		(at 88.9 62.23 0)
-		(effects
-			(font
-				(size 1.27 1.27)
-			)
-			(justify left bottom)
-		)
-	)
-	(label "SDA"
-		(at 158.75 143.51 0)
 		(effects
 			(font
@@
 	(label "MISO_DO"
 		(at 246.38 115.57 0)
-		(effects
-			(font
-				(size 1.27 1.27)
-			)
-			(justify left bottom)
-		)
-	)
-	(label "SCL"
-		(at 158.75 139.7 0)
 		(effects
 			(font
@@
 		(effects
 			(font
-				(size 1.27 1.27)
-			)
-			(justify left bottom)
-		)
-	)
-	(label "MIC_OUT"
-		(at 158.75 130.81 0)
-		(effects
-			(font
