File: kicad_project/_restore_backup_2026-09-08T23-43-19-623/eso32-iot.kicad_sch (KiCad schematic)
At the start: 25 parts, among them J1 B2B-PH-SM4-TB, J2 SS-52400-002, U1 MCP73871

Commit message: update schematic and PCB layout
Parts:
- C1: renamed from C2; footprint Capacitor_SMD:C_0805_2012Metric -> (none)
- C2: renamed from C3; footprint Footprints:T491A -> (none)
- C3: renamed from C4; footprint Footprints:T491A -> (none)
- C4: renamed from C5; footprint Capacitor_SMD:C_0805_2012Metric -> (none)
- C5: renamed from C1; footprint Capacitor_SMD:C_0805_2012Metric -> (none)
- C6: footprint Capacitor_SMD:C_0805_2012Metric -> (none)
- F1: footprint Footprints:FUSC3226X100N -> FUSC3226X100N
- LED1, LED2, LED3, LED4: footprint Footprints:LEDC2012X120N -> LEDC2012X120N
- R1, R10, R2, R3, R4, R5, R6, R7, R8, R9: footprint Resistor_SMD:R_0805_2012Metric -> (none)
Connections:
- net VBUS: no longer J2.A9 (VBUSA2), J2.B9 (VBUSB2)
- net at F1.1, J2.B4 (VBUSB1): no longer C5.2
Other:
- moved on the sheet: C5, F1, J2, R1, R2
