File: kicad_project/_restore_backup_2026-09-08T23-43-19-623/esp32-C3-02.kicad_sch (KiCad schematic)
At the start: 30 parts, among them J3 GSD090012SEU, U2 W25Q32JVSSIQ, U3 ESP32-C3-WROOM-02-H4, U4 CP2102N-Axx-xQFN20, U5 USBLC6-2SC6

Commit message: update schematic and PCB layout
Parts:
- C10, C11, C13, C14, C8: footprint Capacitor_SMD:C_0805_2012Metric -> (none)
- C12, C7, C9: footprint Footprints:T491A -> (none)
- LED5, LED6: footprint Footprints:LEDC2012X120N -> LEDC2012X120N
- R11, R12, R13, R14, R15, R16, R18, R19, R20, R22: footprint Resistor_SMD:R_0805_2012Metric -> (none)
- TP1, TP2, TP3, TP4, TP5: footprint TestPoint:TestPoint_Pad_D1.0mm -> (none)
Connections:
- net DTR renamed DTS
Other:
- sheet User Inteterface ports: added none; removed BOOT, DTR, EN, GPIO18, GPIO19, GPIO8, RTS, SCL, SDA
